Commit message: task A.5 done

File: nuturtle_description/urdf/turtlebot3_burger.urdf.xacro (robot description, xacro)
@@ -3,4 +3,10 @@
     xmlns:xacro="http://ros.org/wiki/xacro">
     <!-- <xacro:include filename="$(find turtlebot3_description)/urdf/common_properties.urdf"/> -->
+    <xacro:property name="props"
+        value="${xacro.load_yaml('$(find nuturtle_description)/config/diff_params.yaml')['/**']['ros__parameters']}" />
+    <xacro:property name="wheel_radius" value="${props['wheel_radius']}" />
+    <xacro:property name="track_width" value="${props['track_width']}" />
+    <xacro:property name="collision_radius" value="${props['collision_radius']}" />
+    <xacro:arg name="color" default="purple" />
     <!-- Init colour -->
     <material name="black">
@@ -34,4 +40,7 @@
         <color rgba="1.0 1.0 1.0 1.0" />
     </material>
+    <material name="purple">
+        <color rgba="0.3 0.16 0.52 1.0" />
+    </material>
     <link name="base_footprint" />
     <joint name="base_joint" type="fixed">
@@ -47,10 +56,15 @@
                     scale="0.001 0.001 0.001" />
             </geometry>
-            <material name="light_black" />
+            <material name="$(arg color)" />
         </visual>
         <collision>
             <origin xyz="-0.032 0 0.070" rpy="0 0 0" />
             <geometry>
-                <box size="0.140 0.140 0.143" />
+                <xacro:if value="${collision_radius &gt; 0}">
+                    <cylinder radius="${collision_radius}" length="0.143" />
+                </xacro:if>
+                <xacro:unless value="${collision_radius &gt; 0}">
+                    <box size="0.140 0.140 0.143" />
+                </xacro:unless>
             </geometry>
         </collision>
@@ -65,5 +79,5 @@
         <parent link="base_link" />
         <child link="wheel_left_link" />
-        <origin xyz="0.0 0.08 0.023" rpy="-1.57 0 0" />
+        <origin xyz="0.0 ${track_width/2} 0.023" rpy="-1.57 0 0" />
         <axis xyz="0 0 1" />
     </joint>
@@ -80,5 +94,5 @@
             <origin xyz="0 0 0" rpy="0 0 0" />
             <geometry>
-                <cylinder length="0.018" radius="0.033" />
+                <cylinder length="0.018" radius="${wheel_radius}" />
             </geometry>
         </collision>
@@ -93,5 +107,5 @@
         <parent link="base_link" />
         <child link="wheel_right_link" />
-        <origin xyz="0.0 -0.080 0.023" rpy="-1.57 0 0" />
+        <origin xyz="0.0 ${-track_width/2} 0.023" rpy="-1.57 0 0" />
         <axis xyz="0 0 1" />
     </joint>
@@ -108,5 +122,5 @@
             <origin xyz="0 0 0" rpy="0 0 0" />
             <geometry>
-                <cylinder length="0.018" radius="0.033" />
+                <cylinder length="0.018" radius="${wheel_radius}" />
             </geometry>
         </collision>
